Commit message: funktioniert jetzt auf dem laptop

File: workspace/ros2_ws/install/mentorpi_description/share/mentorpi_description/urdf/ack.xacro (robot description, xacro)
@@ -1,208 +1 @@
-<?xml version="1.0" ?>
-<robot name="ack" xmlns:xacro="http://ros.org/wiki/xacro">
-    <!-- 瀹氫箟榛戣壊鏉愯川 -->
-  <material name="black">
-    <color rgba="0 0 0 1"/>
-  </material>
-  <!-- 瀹氫箟 base_link -->
-  <link name="base_link">
-    <inertial>
-      <origin rpy="0 0 0" xyz="-0.00186669751054189 3.0253386351986E-05 -0.00605296088229322"/>
-      <mass value="0.0961047465616957"/>
-      <inertia ixx="8.55867486364231E-05" ixy="3.41346959938296E-08" ixz="1.64755227278164E-05" iyy="0.000277248181555496" iyz="-2.95282759133104E-08" izz="0.000344246448853775"/>
-    </inertial>
-    <visual>
-      <origin rpy="0 0 0" xyz="0 0 0"/>
-      <geometry>
-        <mesh filename="package://mentorpi_description/meshes/acker/base_link.STL"/>
-      </geometry>
-      <material name="">
-        <color rgba="1 1 1 1"/>
-      </material>
-    </visual>
-    <collision>
-      <origin rpy="0 0 0" xyz="0 0 0"/>
-      <geometry>
-        <mesh filename="package://mentorpi_description/meshes/acker/base_link.STL"/>
-      </geometry>
-    </collision>
-  </link>
-  <!-- 娣诲姞 base_footprint 閾炬帴 -->
-  <link name="base_footprint"/>
-  <!-- 瀹氫箟 base_footprint 鍒?base_link 鐨勫浐瀹氬叧鑺?-->
-  <joint name="base_footprint_to_base_link" type="fixed">
-    <parent link="base_footprint"/>
-    <child link="base_link"/>
-    <origin xyz="0 0 0.07" rpy="0 0 0"/>
-  </joint>
-  <!-- 瀹氫箟鍏朵粬閾炬帴鍜屽叧鑺?-->
-  <link name="wheel_lf_Link">
-    <inertial>
-      <origin rpy="0 0 0" xyz="1.65897579444685E-06 -0.00270913022688685 -1.5546673051009E-06"/>
-      <mass value="0.0252873083503169"/>
-      <inertia ixx="1.00371783485335E-05" ixy="4.93900109379125E-11" ixz="7.42104604492639E-10" iyy="1.67620175120314E-05" iyz="-5.47583950457701E-11" izz="1.00370342405297E-05"/>
-    </inertial>
-    <visual>
-      <origin rpy="0 0 0" xyz="0 0 0"/>
-      <geometry>
-        <mesh filename="package://mentorpi_description/meshes/acker/wheel_lf_Link.STL"/>
-      </geometry>
-      <material name="">
-        <color rgba="1 1 1 1"/>
-      </material>
-    </visual>
-    <collision>
-      <origin rpy="0 0 0" xyz="0 0 0"/>
-      <geometry>
-        <mesh filename="package://mentorpi_description/meshes/acker/wheel_lf_Link.STL"/>
-      </geometry>
-    </collision>
-  </link>
-  <joint name="wheel_lf_Joint" type="continuous">
-    <origin rpy="0 0 0" xyz="0.06679 0.069739 -0.0288"/>
-    <parent link="base_link"/>
-    <child link="wheel_lf_Link"/>
-    <axis xyz="-2.2918E-05 1 1.9551E-05"/>
-  </joint>
-  <link name="wheel_rf_Link">
-    <inertial>
-      <origin rpy="0 0 0" xyz="-1.48986965733955E-06 0.0027090575018239 1.16299057125596E-06"/>
-      <mass value="0.0252873548617242"/>
-      <inertia ixx="1.00360241846408E-05" ixy="-5.83065201444192E-11" ixz="-8.3023958781985E-11" iyy="1.67622954977732E-05" iyz="6.31638512668579E-11" izz="1.00384960556047E-05"/>
-    </inertial>
-    <visual>
-      <origin rpy="0 0 0" xyz="0 0 0"/>
-      <geometry>
-        <mesh filename="package://mentorpi_description/meshes/acker/wheel_rf_Link.STL"/>
-      </geometry>
-      <material name="">
-        <color rgba="1 1 1 1"/>
-      </material>
-    </visual>
-    <collision>
-      <origin rpy="0 0 0" xyz="0 0 0"/>
-      <geometry>
-        <mesh filename="package://mentorpi_description/meshes/acker/wheel_rf_Link.STL"/>
-      </geometry>
-    </collision>
-  </link>
-  <joint name="wheel_rf_Joint" type="continuous">
-    <origin rpy="0 0 0" xyz="0.066794 -0.069739 -0.028803"/>
-    <parent link="base_link"/>
-    <child link="wheel_rf_Link"/>
-    <axis xyz="-2.2918E-05 1 1.9551E-05"/>
-  </joint>
-  <link name="wheel_lb_Link">
-    <inertial>
-      <origin rpy="0 0 0" xyz="1.62806317080544E-06 -0.00317716794378092 -1.54238045318306E-06"/>
-      <mass value="0.0271078161230754"/>
-      <inertia ixx="1.01056035703468E-05" ixy="4.60479373806495E-11" ixz="7.43896782806142E-10" iyy="1.67990600599721E-05" iyz="-5.763890541079E-11" izz="1.01072652738793E-05"/>
-    </inertial>
-    <visual>
-      <origin rpy="0 0 0" xyz="0 0 0"/>
-      <geometry>
-        <mesh filename="package://mentorpi_description/meshes/acker/wheel_lb_Link.STL"/>
-      </geometry>
-      <material name="">
-        <color rgba="1 1 1 1"/>
-      </material>
-    </visual>
-    <collision>
-      <origin rpy="0 0 0" xyz="0 0 0"/>
-      <geometry>
-        <mesh filename="package://mentorpi_description/meshes/acker/wheel_lb_Link.STL"/>
-      </geometry>
-    </collision>
-  </link>
-  <joint name="wheel_lb_Joint" type="continuous">
-    <origin rpy="0 0 0" xyz="-0.070313 0.07014 -0.027793"/>
-    <parent link="base_link"/>
-    <child link="wheel_lb_Link"/>
-    <axis xyz="-2.2787E-05 1 1.9439E-05"/>
-  </joint>
-  <link name="wheel_rb_Link">
-    <inertial>
-      <origin rpy="0 0 0" xyz="-1.50804700475154E-06 0.00317707027691583 1.18963606317302E-06"/>
-      <mass value="0.0271078005024283"/>
-      <inertia ixx="1.01044417409685E-05" ixy="-5.83069005452564E-11" ixz="-7.56886841840775E-11" iyy="1.67993271276785E-05" iyz="6.31638424138502E-11" izz="1.01087182681654E-05"/>
-    </inertial>
-    <visual>
-      <origin rpy="0 0 0" xyz="0 0 0"/>
-      <geometry>
-        <mesh filename="package://mentorpi_description/meshes/acker/wheel_rb_Link.STL"/>
-      </geometry>
-      <material name="">
-        <color rgba="1 1 1 1"/>
-      </material>
-    </visual>
-    <collision>
-      <origin rpy="0 0 0" xyz="0 0 0"/>
-      <geometry>
-        <mesh filename="package://mentorpi_description/meshes/acker/wheel_rb_Link.STL"/>
-      </geometry>
-          </collision>
-  </link>
-  <joint name="wheel_rb_Joint" type="continuous">
-    <origin rpy="0 0 0" xyz="-0.07031 -0.07014 -0.027796"/>
-    <parent link="base_link"/>
-    <child link="wheel_rb_Link"/>
-    <axis xyz="-2.2787E-05 1 1.9439E-05"/>
-  </joint>
-  <link name="depth_cam">
-    <inertial>
-      <origin rpy="0 0 0" xyz="0.0023402290651429 0.00113784597946548 -0.0102127064032341"/>
-      <mass value="0.0270474748429678"/>
-      <inertia ixx="1.43718505822118E-05" ixy="1.24779382573379E-07" ixz="1.29836477956744E-08" iyy="1.65912768209848E-06" iyz="2.28291478579102E-08" izz="1.45615925510082E-05"/>
-    </inertial>
-    <visual>
-      <origin rpy="0 0 0" xyz="0 0 0"/>
-      <geometry>
-        <mesh filename="package://mentorpi_description/meshes/acker/cam_Link.STL"/>
-      </geometry>
-      <material name="">
-        <color rgba="1 1 1 1"/>
-      </material>
-    </visual>
-    <collision>
-      <origin rpy="0 0 0" xyz="0 0 0"/>
-      <geometry>
-        <mesh filename="package://mentorpi_description/meshes/acker/cam_Link.STL"/>
-      </geometry>
-    </collision>
-  </link>
-  <joint name="cam_Joint" type="fixed">
-    <origin rpy="0 0 0" xyz="0.064015 -0.00013463 0.051155"/>
-    <parent link="base_link"/>
-    <child link="depth_cam"/>
-    <axis xyz="0 0 0"/>
-  </joint>
-  <link name="lidar_frame">
-    <inertial>
-      <origin rpy="0 0 0" xyz="8.65086433231368E-05 9.02624784523964E-05 -0.0183546134614858"/>
-      <mass value="0.0405423044068563"/>
-      <inertia ixx="4.98470776877503E-06" ixy="-1.54076264166869E-07" ixz="2.05182706824286E-09" iyy="5.03926730822203E-06" iyz="1.1006285118993E-08" izz="8.25645669548359E-06"/>
-    </inertial>
-    <visual>
-      <origin rpy="0 0 0" xyz="0 0 0"/>
-      <geometry>
-        <mesh filename="package://mentorpi_description/meshes/acker/lidar_Link.STL"/>
-      </geometry>
-      <material name="">
-        <color rgba="1 1 1 1"/>
-      </material>
-    </visual>
-    <collision>
-      <origin rpy="0 0 0" xyz="0 0 0"/>
-      <geometry>
-        <mesh filename="package://mentorpi_description/meshes/acker/lidar_Link.STL"/>
-      </geometry>
-    </collision>
-  </link>
-  <joint name="lidar_Joint" type="fixed">
-    <origin rpy="0 0 0" xyz="-0.0096019 -8.533E-05 0.092501"/>
-    <parent link="base_link"/>
-    <child link="lidar_frame"/>
-    <axis xyz="0 0 0"/>
-  </joint>
-  <xacro:include filename="$(find mentorpi_description)/urdf/imu.urdf.xacro"/>
-</robot>
+/home/oli/Desktop/Oliver/Uni/MA/RepoTrajektorienfolgeregelung/MA-Trajektorienfolgeregelung/workspace/ros2_ws/build/mentorpi_description/urdf/ack.xacro

File: workspace/ros2_ws/install/mentorpi_description/share/mentorpi_description/urdf/imu.urdf.xacro (robot description, xacro)
@@ -1,20 +1 @@
-<?xml version="1.0" encoding="utf-8"?>
-<robot name="imu" xmlns:xacro="http://ros.org/wiki/xacro">
-  <xacro:property name="M_PI" value="3.1415926535897931"/>
-  <link
-    name="imu_link">
-  </link>
-  <joint
-    name="imu_joint"
-    type="fixed">
-    <origin
-      xyz="0 0 ${0.025 - 0.0295 + 0.0965/2 + 0.0678410821576746}"
-      rpy="0 0 ${-M_PI/2}" />
-    <parent
-      link="base_link" />
-    <child
-      link="imu_link" />
-    <axis
-      xyz="0 0 0" />
-  </joint>
-</robot>
+/home/oli/Desktop/Oliver/Uni/MA/RepoTrajektorienfolgeregelung/MA-Trajektorienfolgeregelung/workspace/ros2_ws/build/mentorpi_description/urdf/imu.urdf.xacro

File: workspace/ros2_ws/install/mentorpi_description/share/mentorpi_description/urdf/inertial_matrix.xacro (robot description, xacro)
@@ -1,44 +1 @@
-<?xml version="1.0" encoding="utf-8"?>
-<robot name="inertial_matrix" xmlns:xacro="http://ros.org/wiki/xacro">
-  <xacro:property name="M_PI" value="3.1415926535897931" />
-  <!-- Macro for inertia matrix -->
-  <xacro:macro name="sphere_inertial" params="m r">
-    <inertial>
-      <mass value="${m}" />
-      <inertia
-        ixx="${2*m*r*r/5}"
-        ixy="0"
-        ixz="0"
-        iyy="${2*m*r*r/5}"
-        iyz="0"
-        izz="${2*m*r*r/5}" />
-    </inertial>
-  </xacro:macro>
-  <xacro:macro name="cylinder_inertial" params="m r h">
-    <inertial>
-      <mass value="${m}" />
-      <inertia
-        ixx="${m*(3*r*r+h*h)/12}"
-        ixy = "0"
-        ixz = "0"
-        iyy="${m*(3*r*r+h*h)/12}"
-        iyz = "0"
-        izz="${m*r*r/2}" />
-    </inertial>
-  </xacro:macro>
-  <xacro:macro name="box_inertial" params="m w h d x y z">
-      <inertial>
-      <origin
-        xyz="${x} ${y} ${z}"
-        rpy="0 0 0" />
-      <mass value="${m}" />
-      <inertia
-        ixx="${m*(h*h+d*d)/12}"
-        ixy = "0"
-        ixz = "0"
-        iyy="${m*(w*w+d*d)/12}"
-        iyz = "0"
-        izz="${m*(w*w+h*h)/12}" />
-    </inertial>
-  </xacro:macro>
-</robot>
+/home/oli/Desktop/Oliver/Uni/MA/RepoTrajektorienfolgeregelung/MA-Trajektorienfolgeregelung/workspace/ros2_ws/build/mentorpi_description/urdf/inertial_matrix.xacro

File: workspace/ros2_ws/install/mentorpi_description/share/mentorpi_description/urdf/lidar.urdf.xacro (robot description, xacro)
@@ -1,12 +1 @@
-<?xml version="1.0" encoding="utf-8"?>
-<robot name="lidar_a1" xmlns:xacro="http://ros.org/wiki/xacro" >
-  <xacro:property name="M_PI" value="3.1415926535897931"/>
-  <link name="lidar_frame" />
-  <joint
-    name="lidar_frame"
-    type="fixed">
-    <origin xyz="0 0 0" rpy="0 0 ${M_PI}" />
-    <parent link="lidar_link" />
-    <child link="lidar_frame" />
-  </joint>
-</robot>
+/home/oli/Desktop/Oliver/Uni/MA/RepoTrajektorienfolgeregelung/MA-Trajektorienfolgeregelung/workspace/ros2_ws/build/mentorpi_description/urdf/lidar.urdf.xacro

File: workspace/ros2_ws/install/mentorpi_description/share/mentorpi_description/urdf/materials.xacro (robot description, xacro)
@@ -1,27 +1 @@
-<?xml version="1.0"?>
-<robot name="material" xmlns:xacro="http://ros.org/wiki/xacro">
-    <material name="black">
-        <color rgba="0.1 0.1 0.1 1.0"/>
-    </material>
-    <material name="blue">
-        <color rgba="0.0 0.0 0.8 1.0"/>
-    </material>
-    <material name="green">
-        <color rgba="0.4 0.9 0.4 1.0"/>
-    </material>
-    <material name="gray">
-        <color rgba="0.7 0.7 0.7 1.0"/>
-    </material>
-    <material name="darkgray">
-        <color rgba="0.3 0.3 0.3 1.0"/>
-    </material>
-    <material name="red">
-        <color rgba="0.8 0.0 0.0 1.0"/>
-    </material>
-    <material name="white">
-        <color rgba="1.0 1.0 1.0 1.0"/>
-    </material>
-    <material name="yellow">
-        <color rgba="0.8 0.8 0.0 1.0"/>
-    </material>
-</robot>
+/home/oli/Desktop/Oliver/Uni/MA/RepoTrajektorienfolgeregelung/MA-Trajektorienfolgeregelung/workspace/ros2_ws/build/mentorpi_description/urdf/materials.xacro

File: workspace/ros2_ws/install/mentorpi_description/share/mentorpi_description/urdf/mecanum.xacro (robot description, xacro)
@@ -1,209 +1 @@
-<?xml version="1.0" ?>
-<robot name="mecanum" xmlns:xacro="http://ros.org/wiki/xacro">
-  <!-- 定义黑色材质 -->
-  <material name="black">
-    <color rgba="0 0 0 1"/>
-  </material>
-  <link name="imu_link"/>
-  <joint name="imu_joint" type="fixed">
-    <parent link="base_link"/>
-    <child link="imu_link"/>
-    <origin xyz="0 0 0" rpy="0 0 -1.57"/>
-  </joint>
-  <link name="base_footprint"/>
-  <joint name="base_footprint_to_base_link" type="fixed">
-    <parent link="base_footprint"/>
-    <child link="base_link"/>
-    <origin xyz="0 0 0.07" rpy="0 0 0"/>
-  </joint>
-  <link name="base_link">
-    <inertial>
-      <origin rpy="0 0 0" xyz="7.82634169708696E-05 3.66518389137982E-05 0.0068167426737893"/>
-      <mass value="0.080358044299185"/>
-      <inertia ixx="9.92047502462735E-05" ixy="3.20099144678921E-08" ixz="1.15869166655817E-05" iyy="0.000292461515602123" iyz="-2.92890751882614E-08" izz="0.000367604260834833"/>
-    </inertial>
-    <visual>
-      <origin rpy="0 0 0" xyz="0 0 0"/>
-      <geometry>
-        <mesh filename="package://mentorpi_description/meshes/mecanum/base_link.STL"/>
-      </geometry>
-      <material name="">
-        <color rgba="1 1 1 1"/>
-      </material>
-    </visual>
-    <collision>
-      <origin rpy="0 0 0" xyz="0 0 0"/>
-      <geometry>
-        <mesh filename="package://mentorpi_description/meshes/mecanum/base_link.STL"/>
-      </geometry>
-    </collision>
-  </link>
-  <link name="wheel_lf_Link">
-    <inertial>
-      <origin rpy="0 0 0" xyz="6.23194347770945E-05 -0.00574614971695361 2.98597149463314E-05"/>
-      <mass value="0.0378743634664218"/>
-      <inertia ixx="3.67678518315829E-06" ixy="-1.42189561270372E-09" ixz="-1.20320324868622E-08" iyy="5.81008995754212E-06" iyz="1.72329758812212E-09" izz="3.67939460898329E-06"/>
-    </inertial>
-    <visual>
-      <origin rpy="0 0 0" xyz="0 0 0"/>
-      <geometry>
-        <mesh filename="package://mentorpi_description/meshes/mecanum/wheel_lf_Link.STL"/>
-      </geometry>
-      <material name="">
-        <color rgba="1 1 1 1"/>
-      </material>
-    </visual>
-    <collision>
-      <origin rpy="0 0 0" xyz="0 0 0"/>
-      <geometry>
-        <mesh filename="package://mentorpi_description/meshes/mecanum/wheel_lf_Link.STL"/>
-      </geometry>
-    </collision>
-  </link>
-  <joint name="wheel_lf_Joint" type="continuous">
-    <origin rpy="0 0 0" xyz="0.067052 0.07591 -0.018408"/>
-    <parent link="base_link"/>
-    <child link="wheel_lf_Link"/>
-    <axis xyz="0.00012228 1 -4.0642E-05"/>
-  </joint>
-  <link name="wheel_rf_Link">
-    <inertial>
-      <origin rpy="0 0 0" xyz="6.22118237483121E-05 0.00574626671891662 2.98167804906255E-05"/>
-      <mass value="0.0378687944527435"/>
-      <inertia ixx="3.67635322071944E-06" ixy="1.49075106320551E-09" ixz="-1.20440562033349E-08" iyy="5.80905053329656E-06" iyz="-1.7316728972649E-09" izz="3.67859542953002E-06"/>
-    </inertial>
-    <visual>
-      <origin rpy="0 0 0" xyz="0 0 0"/>
-      <geometry>
-        <mesh filename="package://mentorpi_description/meshes/mecanum/wheel_rf_Link.STL"/>
-      </geometry>
-      <material name="">
-        <color rgba="1 1 1 1"/>
-      </material>
-    </visual>
-    <collision>
-      <origin rpy="0 0 0" xyz="0 0 0"/>
-      <geometry>
-        <mesh filename="package://mentorpi_description/meshes/mecanum/wheel_rf_Link.STL"/>
-      </geometry>
-    </collision>
-  </link>
-  <joint name="wheel_rf_Joint" type="continuous">
-    <origin rpy="0 0 0" xyz="0.067052 -0.07591 -0.018408"/>
-    <parent link="base_link"/>
-    <child link="wheel_rf_Link"/>
-    <axis xyz="0.00012228 1 -4.0642E-05"/>
-  </joint>
-  <link name="wheel_lb_Link">
-    <inertial>
-      <origin rpy="0 0 0" xyz="-4.39089176767909E-05 -0.00574629427498616 3.59684108433914E-05"/>
-      <mass value="0.0378689402752074"/>
-      <inertia ixx="3.67629328541386E-06" ixy="1.48552620491244E-09" ixz="1.20977149812926E-08" iyy="5.80903210056483E-06" iyz="1.72555302795062E-09" izz="3.6786318488588E-06"/>
-    </inertial>
-    <visual>
-      <origin rpy="0 0 0" xyz="0 0 0"/>
-      <geometry>
-        <mesh filename="package://mentorpi_description/meshes/mecanum/wheel_lb_Link.STL"/>
-      </geometry>
-      <material name="">
-        <color rgba="1 1 1 1"/>
-      </material>
-    </visual>
-    <collision>
-      <origin rpy="0 0 0" xyz="0 0 0"/>
-      <geometry>
-        <mesh filename="package://mentorpi_description/meshes/mecanum/wheel_lb_Link.STL"/>
-      </geometry>
-    </collision>
-  </link>
-  <joint name="wheel_lb_Joint" type="continuous">
-    <origin rpy="0 0 0" xyz="-0.06764 0.07591 -0.018414"/>
-    <parent link="base_link"/>
-    <child link="wheel_lb_Link"/>
-    <axis xyz="0 1 0"/>
-  </joint>
-  <link name="wheel_rb_Link">
-    <inertial>
-      <origin rpy="0 0 0" xyz="-6.2256559793028E-05 0.00574614092169209 2.96857054536206E-05"/>
-      <mass value="0.0378742388937267"/>
-      <inertia ixx="3.67690880733038E-06" ixy="-1.42614754024296E-09" ixz="1.19925568848388E-08" iyy="5.81009054149328E-06" iyz="-1.72488948912739E-09" izz="3.67928241656151E-06"/>
-    </inertial>
-    <visual>
-      <origin rpy="0 0 0" xyz="0 0 0"/>
-      <geometry>
-        <mesh filename="package://mentorpi_description/meshes/mecanum/wheel_rb_Link.STL"/>
-      </geometry>
-      <material name="">
-        <color rgba="1 1 1 1"/>
-      </material>
-    </visual>
-    <collision>
-      <origin rpy="0 0 0" xyz="0 0 0"/>
-      <geometry>
-        <mesh filename="package://mentorpi_description/meshes/mecanum/wheel_rb_Link.STL"/>
-      </geometry>
-    </collision>
-  </link>
-  <joint name="wheel_rb_Joint" type="continuous">
-    <origin rpy="0 0 0" xyz="-0.067621 -0.07591 -0.018408"/>
-    <parent link="base_link"/>
-    <child link="wheel_rb_Link"/>
-    <axis xyz="0 1 0"/>
-  </joint>
-  <link name="depth_cam">
-    <inertial>
-      <origin rpy="0 0 0" xyz="0.0023402290706885 0.00113784597175737 -0.010212706399263"/>
-      <mass value="0.0270474748712619"/>
-      <inertia ixx="1.43718505980935E-05" ixy="1.24779390700312E-07" ixz="1.29836475580818E-08" iyy="1.65912768335363E-06" iyz="2.28291474116005E-08" izz="1.45615925671284E-05"/>
-    </inertial>
-    <visual>
-      <origin rpy="0 0 0" xyz="0 0 0"/>
-      <geometry>
-        <mesh filename="package://mentorpi_description/meshes/mecanum/cam_Link.STL"/>
-      </geometry>
-      <material name="">
-        <color rgba="1 1 1 1"/>
-      </material>
-    </visual>
-    <collision>
-      <origin rpy="0 0 0" xyz="0 0 0"/>
-      <geometry>
-        <mesh filename="package://mentorpi_description/meshes/mecanum/cam_Link.STL"/>
-      </geometry>
-    </collision>
-  </link>
-  <joint name="cam_Joint" type="fixed">
-    <origin rpy="0 0 0" xyz="0.061376 -0.00013463 0.051154"/>
-    <parent link="base_link"/>
-    <child link="depth_cam"/>
-    <axis xyz="0 0 0"/>
-  </joint>
-  <link name="lidar_frame">
-    <inertial>
-      <origin rpy="0 0 0" xyz="8.65086404290248E-05 9.02624664517182E-05 -0.0183546134707293"/>
-      <mass value="0.0405423044439003"/>
-      <inertia ixx="4.98470777040832E-06" ixy="-1.5407626531037E-07" ixz="2.05182756187779E-09" iyy="5.03926730954594E-06" iyz="1.10062857837226E-08" izz="8.25645669795306E-06"/>
-    </inertial>
-    <visual>
-      <origin rpy="0 0 0" xyz="0 0 0"/>
-      <geometry>
-        <mesh filename="package://mentorpi_description/meshes/mecanum/lidar_Link.STL"/>
-      </geometry>
-      <material name="">
-        <color rgba="1 1 1 1"/>
-      </material>
-    </visual>
-    <collision>
-      <origin rpy="0 0 0" xyz="0 0 0"/>
-      <geometry>
-        <mesh filename="package://mentorpi_description/meshes/mecanum/lidar_Link.STL"/>
-      </geometry>
-    </collision>
-  </link>
-  <joint name="lidar_Joint" type="fixed">
-    <origin rpy="0 0 0" xyz="-0.012242 -8.533E-05 0.092501"/>
-    <parent link="base_link"/>
-    <child link="lidar_frame"/>
-    <axis xyz="0 0 0"/>
-  </joint>
-</robot>
+/home/oli/Desktop/Oliver/Uni/MA/RepoTrajektorienfolgeregelung/MA-Trajektorienfolgeregelung/workspace/ros2_ws/build/mentorpi_description/urdf/mecanum.xacro

File: workspace/ros2_ws/install/mentorpi_description/share/mentorpi_description/urdf/mentorpi.xacro (robot description, xacro)
@@ -1,11 +1 @@
-<?xml version="1.0" encoding="utf-8"?>
-<robot name="rosmentor" xmlns:xacro="http://ros.org/wiki/xacro">
-    <xacro:property name="machine"      value="$(env MACHINE_TYPE)"/>
-    <xacro:if value="${machine == 'MentorPi_Mecanum'}">
-        <xacro:include filename="$(find mentorpi_description)/urdf/mecanum.xacro"/>
-    </xacro:if>
-    <xacro:if value="${machine == 'MentorPi_Acker'}">
-        <xacro:include filename="$(find mentorpi_description)/urdf/ack.xacro"/>
-    </xacro:if>
-    <xacro:include filename="$(find mentorpi_description)/urdf/inertial_matrix.xacro" />
-</robot>
+/home/oli/Desktop/Oliver/Uni/MA/RepoTrajektorienfolgeregelung/MA-Trajektorienfolgeregelung/workspace/ros2_ws/build/mentorpi_description/urdf/mentorpi.xacro
